Commit message: Torso as origin point

File: body.urdf (robot description, URDF)
Before this commit: robot robot, 3 links, 2 joints
Links:
- removed link Arm
- removed link Leg
- added link BackLeg, mass 1; collision box size=1 1 1; visual box size=1 1 1
- added link FrontLeg, mass 1; collision box size=1 1 1; visual box size=1 1 1
Joints:
- removed joint Leg_Arm
- removed joint Torso_Leg
- added joint Torso_BackLeg: type revolute, parent Torso, child BackLeg, origin xyz=0.5 0 1 rpy=0 0 0, axis 0 1 0, limit lower=-3.14159 upper=3.14159 effort=0.0 velocity=0.0
- added joint Torso_FrontLeg: type revolute, parent Torso, child FrontLeg, origin xyz=1.5 0 1 rpy=0 0 0, axis 0 1 0, limit lower=-3.14159 upper=3.14159 effort=0.0 velocity=0.0

Commit message: changes

File: body.urdf (robot description, URDF)
Before this commit: robot robot, 3 links, 2 joints
Joints:
- joint Torso_BackLeg: origin xyz=0.5 0 1 rpy=0 0 0 -> xyz=0.5 0 2 rpy=0 0 0

Commit message: changes

File: body.urdf (robot description, URDF)
Before this commit: robot robot, 3 links, 2 joints
Joints:
- joint Torso_BackLeg: origin xyz=0.5 0 2 rpy=0 0 0 -> xyz=0.5 0 1 rpy=0 0 0

Commit message: Working quadrupede

File: body.urdf (robot description, URDF)
Before this commit: robot robot, 3 links, 2 joints
Links:
- added link BackLowerLeg, mass 1; collision box size=0.2 0.2 1; visual box size=0.2 0.2 1
- added link FrontLowerLeg, mass 1; collision box size=0.2 0.2 1; visual box size=0.2 0.2 1
- added link LeftLeg, mass 1; collision box size=1 0.2 0.2; visual box size=1 0.2 0.2
- added link LeftLowerLeg, mass 1; collision box size=0.2 0.2 1; visual box size=0.2 0.2 1
- added link RightLeg, mass 1; collision box size=1 0.2 0.2; visual box size=1 0.2 0.2
- added link RightLowerLeg, mass 1; collision box size=0.2 0.2 1; visual box size=0.2 0.2 1
- link BackLeg: geometry collision box size=0.2 1 0.2; visual box size=0.2 1 0.2
- link FrontLeg: geometry collision box size=0.2 1 0.2; visual box size=0.2 1 0.2
Joints:
- added joint BackLeg_BackLowerLeg: type revolute, parent BackLeg, child BackLowerLeg, origin xyz=0 -1 0 rpy=0 0 0, axis 1 0 0, limit lower=-3.14159 upper=3.14159 effort=0.0 velocity=0.0
- added joint FrontLeg_FrontLowerLeg: type revolute, parent FrontLeg, child FrontLowerLeg, origin xyz=0 1 0 rpy=0 0 0, axis 1 0 0, limit lower=-3.14159 upper=3.14159 effort=0.0 velocity=0.0
- added joint LeftLeg_LeftLowerLeg: type revolute, parent LeftLeg, child LeftLowerLeg, origin xyz=-1 0 0 rpy=0 0 0, axis 0 1 0, limit lower=-3.14159 upper=3.14159 effort=0.0 velocity=0.0
- added joint RightLeg_RightLowerLeg: type revolute, parent RightLeg, child RightLowerLeg, origin xyz=1 0 0 rpy=0 0 0, axis 0 1 0, limit lower=-3.14159 upper=3.14159 effort=0.0 velocity=0.0
- added joint Torso_LeftLeg: type revolute, parent Torso, child LeftLeg, origin xyz=-0.5 0 1 rpy=0 0 0, axis 0 1 0, limit lower=-3.14159 upper=3.14159 effort=0.0 velocity=0.0
- added joint Torso_RightLeg: type revolute, parent Torso, child RightLeg, origin xyz=0.5 0 1 rpy=0 0 0, axis 0 1 0, limit lower=-3.14159 upper=3.14159 effort=0.0 velocity=0.0
- joint Torso_BackLeg: axis 0 1 0 -> 1 0 0; origin xyz=0.5 0 1 rpy=0 0 0 -> xyz=0 -0.5 1 rpy=0 0 0
- joint Torso_FrontLeg: axis 0 1 0 -> 1 0 0; origin xyz=1.5 0 1 rpy=0 0 0 -> xyz=0 0.5 1 rpy=0 0 0

Commit message: many changes

File: body.urdf (robot description, URDF)
Before this commit: robot robot, 9 links, 8 joints
Links:
- removed link BackLeg
- removed link BackLowerLeg
- removed link FrontLeg
- removed link FrontLowerLeg
- removed link LeftLeg
- removed link LeftLowerLeg
- removed link RightLeg
- removed link RightLowerLeg
- removed link Torso
- added link Link0, mass 1; collision box size=1 1 1; visual box size=1 1 1
- added link Link1, mass 1; collision box size=2.6693821361734678 0.4327616018632101 1.7711267594879887; visual box size=2.6693821361734678 0.4327616018632101 1.7711267594879887
- added link Link2, mass 1; collision box size=0.759066480266209 2.8889208543379343 1.0049235675457666; visual box size=0.759066480266209 2.8889208543379343 1.0049235675457666
- added link Link3, mass 1; collision box size=0.4082961299083917 2.251485945013828 0.2940264216787285; visual box size=0.4082961299083917 2.251485945013828 0.2940264216787285
- added link Link4, mass 1; collision box size=0.8183941373261797 1.3936861445493238 1.444172760135227; visual box size=0.8183941373261797 1.3936861445493238 1.444172760135227
Joints:
- removed joint BackLeg_BackLowerLeg
- removed joint FrontLeg_FrontLowerLeg
- removed joint LeftLeg_LeftLowerLeg
- removed joint RightLeg_RightLowerLeg
- removed joint Torso_BackLeg
- removed joint Torso_FrontLeg
- removed joint Torso_LeftLeg
- removed joint Torso_RightLeg
- added joint Link0_Link1: type revolute, parent Link0, child Link1, origin xyz=0 -0.5 2.6467904985695294 rpy=0 0 0, axis 0 1 0, limit lower=-3.14159 upper=3.14159 effort=0.0 velocity=0.0
- added joint Link1_Link2: type revolute, parent Link1, child Link2, origin xyz=0.2819731415156157 -1.0622214044388734 -0.8855633797439943 rpy=0 0 0, axis 0 1 0, limit lower=-3.14159 upper=3.14159 effort=0.0 velocity=0.0
- added joint Link2_Link3: type revolute, parent Link2, child Link3, origin xyz=-0.3795332401331045 0.6885085974579028 -0.5011749405924517 rpy=0 0 0, axis 0 1 0, limit lower=-3.14159 upper=3.14159 effort=0.0 velocity=0.0
- added joint Link3_Link4: type revolute, parent Link3, child Link4, origin xyz=-1.1920359920542152 1.125742972506914 -0.037965798165469855 rpy=0 0 0, axis 0 1 0, limit lower=-3.14159 upper=3.14159 effort=0.0 velocity=0.0

Commit message: useless changes

File: body.urdf (robot description, URDF)
Before this commit: robot robot, 5 links, 4 joints
Links:
- added link Link5, mass 1; collision box size=0.9472195273574695 0.6409862941380853 0.9602051915759192; visual box size=0.9472195273574695 0.6409862941380853 0.9602051915759192
- added link Link6, mass 1; collision box size=0.5634558816959845 0.09783053984229151 0.17626100186217541; visual box size=0.5634558816959845 0.09783053984229151 0.17626100186217541
- added link Link7, mass 1; collision box size=0.3911111312671208 0.5576946974074953 0.7159794715821339; visual box size=0.3911111312671208 0.5576946974074953 0.7159794715821339
- added link Link8, mass 1; collision box size=0.6501964118114348 0.18600455669371163 0.24930573297803094; visual box size=0.6501964118114348 0.18600455669371163 0.24930573297803094
- added link Link9, mass 1; collision box size=0.36491099332142596 0.2652942543331973 0.8161144436561504; visual box size=0.36491099332142596 0.2652942543331973 0.8161144436561504
- link Link1: geometry collision box size=0.09969996298241957 0.4248765394737186 0.42012055230878254; visual box size=0.09969996298241957 0.4248765394737186 0.42012055230878254
- link Link2: geometry collision box size=0.15842796956633853 0.06189328384976567 0.4719639805808479; visual box size=0.15842796956633853 0.06189328384976567 0.4719639805808479
- link Link3: geometry collision box size=0.987290029128502 0.8214684144606286 0.3626316309803145; visual box size=0.987290029128502 0.8214684144606286 0.3626316309803145
- link Link4: geometry collision box size=0.984278777486368 0.5703215308521559 0.17735400341067753; visual box size=0.984278777486368 0.5703215308521559 0.17735400341067753
Joints:
- added joint Link4_Link5: type revolute, parent Link4, child Link5, origin xyz=0.35658155936555963 -0.13912019885096794 0.08867700170533876 rpy=0 0 0, axis 0 1 0, limit lower=-3.14159 upper=3.14159 effort=0.0 velocity=0.0
- added joint Link5_Link6: type revolute, parent Link5, child Link6, origin xyz=0.47360976367873475 0.256098540549326 0.8423197766439294 rpy=0 0 0, axis 0 1 0, limit lower=-3.14159 upper=3.14159 effort=0.0 velocity=0.0
- added joint Link6_Link7: type revolute, parent Link6, child Link7, origin xyz=0.26576963585502045 -0.006592732595785571 -0.08813050093108771 rpy=0 0 0, axis 0 1 0, limit lower=-3.14159 upper=3.14159 effort=0.0 velocity=0.0
- added joint Link7_Link8: type revolute, parent Link7, child Link8, origin xyz=0.06727437752968368 0.27884734870374767 -0.3429069207224981 rpy=0 0 0, axis 0 1 0, limit lower=-3.14159 upper=3.14159 effort=0.0 velocity=0.0
- added joint Link8_Link9: type revolute, parent Link8, child Link9, origin xyz=0.26863692631272035 0.18600455669371163 0.05148310294216213 rpy=0 0 0, axis 0 1 0, limit lower=-3.14159 upper=3.14159 effort=0.0 velocity=0.0
- joint Link0_Link1: origin xyz=0 -0.5 2.6467904985695294 rpy=0 0 0 -> xyz=0 0.5 1.7674990226569443 rpy=0 0 0
- joint Link1_Link2: origin xyz=0.2819731415156157 -1.0622214044388734 -0.8855633797439943 rpy=0 0 0 -> xyz=0.04984998149120978 -0.00011154876547950221 0.04385371872456739 rpy=0 0 0
- joint Link2_Link3: origin xyz=-0.3795332401331045 0.6885085974579028 -0.5011749405924517 rpy=0 0 0 -> xyz=0.18222563423572458 0.021502885182580846 -0.23598199029042394 rpy=0 0 0
- joint Link3_Link4: origin xyz=-1.1920359920542152 1.125742972506914 -0.037965798165469855 rpy=0 0 0 -> xyz=0.493645014564251 0.36840326681148117 -0.32005598004563807 rpy=0 0 0
